Commit message: URDF: raiz sem massa (base_footprint) e o exit code -2 documentado
O teste de campo do tutorial trouxe dois achados.

1) Erro meu. O base_link tinha <inertial> e era a raiz, o que faz o
   robot_state_publisher avisar:

     WARN kdl_parser: The root link base_link has an inertia specified in
     the URDF, but KDL does not support a root link with an inertia.

   Nao quebra nada -- o robo aparece e a TF funciona --, mas apareceria para
   todo aluno. A saida que o proprio aviso sugere e a convencao da area, e e
   ela que o exemplo passa a usar: um base_footprint vazio na raiz, ligado ao
   base_link por junta fixa, com a altura do robo escrita explicitamente no
   origin (0.09 = raio da roda + o quanto a roda desce da base).

   Ganho alem de calar o aviso: base_footprint/base_link e o par que o Nav2 e
   o SLAM esperam no TP3. Um robo que navega precisa saber onde toca o chao,
   nao so onde fica o centro da carcaca. Secao propria no tutorial explicando
   as duas razoes.

   O Fixed Frame do .rviz e as citacoes de raiz no tutorial e no README foram
   atualizados junto. URDF revalidado por script, agora tambem conferindo que
   a raiz nao tem <inertial>.

2) Ruido com cara de falha. Ao dar Ctrl+C:

     [ERROR] joint_state_publisher_gui: process has died [exit code -2]
     [INFO]  robot_state_publisher: process has finished cleanly
     [INFO]  rviz2: process has finished cleanly

   Codigo de saida NEGATIVO significa terminado por sinal, e -2 e o sinal 2,
   o proprio SIGINT do Ctrl+C. O processo obedeceu. O joint_state_publisher_gui
   e uma janela Qt e nao instala tratador de SIGINT que saia com zero, entao o
   launch classifica como ERROR um encerramento normal.

   Mesma familia do 'Exception ignored in: Future.__del__' da Aula 3, e a
   licao generaliza: [ERROR] no launch nao significa que algo falhou -- ele
   classifica por codigo de saida, e sair por sinal da codigo negativo.

File: exemplos/aula09-urdf/meu_robo_description/urdf/meu_robo.urdf (robot description, URDF)
Before this commit: robot meu_robo, 6 links, 5 joints
Links:
- added link base_footprint
Joints:
- added joint junta_base: type fixed, parent base_footprint, child base_link, origin xyz=0 0 0.09 rpy=0 0 0
